File: PCB/revo-main/revo-main.kicad_sch (KiCad schematic)
At the start: 58 parts, among them J10 DS5180, J12 SERVO CONN, J13 KF301-2P, J14 KF301-2P, J15 BUZZER, J16 KF301-2P, J17 E-STOP, J19 KF301-2P, J20 JST_2mm_LiPo, J21 XT60-M, J24 FAN PWR, J26 Conn, J28 3V3, J29 I2C, J34 Conn, J35 Conn, J4 JST_2mm_LiPo, J5 JST_2mm_LiPo, J6 JST_2mm_LiPo, J7 JST_2mm_LiPo, J8 DS5180, J9 DS5180, Q2 2N7002, Q3 AOD4185, Q4 BSS138, SW1 Home, U1 HT7350, U10 INA219AxD, U6 INA219AxD, U9 INA219AxD, X1 Power

Commit message: init
Parts:
- D2: Availability In Stock -> (none); Package None -> (none); Price None -> (none)
- R21: MPN (none) -> 13-MFR50SFTE52-2K2CT-ND
